Commit message: baker

File: maccepa_description/gazebo/gazebo.urdf.xacro (robot description, xacro)
@@ -2,12 +2,11 @@
 <robot>
     <gazebo>
-        <!--<plugin filename="libgazebo_ros_control.so" name="ros_control">-->
-            <!--<robotNamespace>/maccepa</robotNamespace>-->
-        <!--</plugin>-->
-        <plugin name="maccepa_shoulder" filename="libmaccepa_plugin.so">
+        <plugin filename="libgazebo_ros_control.so" name="ros_control">
+            <robotNamespace>/maccepa</robotNamespace>
+        </plugin>
+        <plugin filename="libmaccepa_plugin.so" name="maccepa_shoulder">
             <joint>shoulder</joint>
-            <command_topic>/shoulder/command</command_topic>
-            <stiffness_topic>/shoulder/stiffness</stiffness_topic>
-            <pos_topic>/shoulder/position</pos_topic>
+            <cardioid_motor_command_topic>/maccepa_plugin/shoulder/cardioid_motor/command</cardioid_motor_command_topic>
+            <pretension_motor_command_topic>/maccepa_plugin/shoulder/pretension_motor/command</pretension_motor_command_topic>
             <!-- Maccepa 2.0 parameters BEGIN -->
             <k>3742</k><!-- [N/m] spring constant -->
@@ -17,11 +16,10 @@
             <R_pretension>0.01</R_pretension><!-- [m] motor 2 spool radius -->
             <!-- Maccepa 2.0 parameters END -->
-            <joint_motor>shoulder_motor_joint</joint_motor>
+            <cardioid_motor_joint>shoulder_motor_joint</cardioid_motor_joint>
         </plugin>
-        <plugin name="maccepa_elbow" filename="libmaccepa_plugin.so">
+        <plugin filename="libmaccepa_plugin.so" name="maccepa_elbow">
             <joint>elbow</joint>
-            <command_topic>/elbow/command</command_topic>
-            <stiffness_topic>/elbow/stiffness</stiffness_topic>
-            <pos_topic>/elbow/position</pos_topic>
+            <cardioid_motor_command_topic>/maccepa_plugin/elbow/cardioid_motor/command</cardioid_motor_command_topic>
+            <pretension_motor_command_topic>/maccepa_plugin/elbow/pretension_motor/command</pretension_motor_command_topic>
             <!-- Maccepa 2.0 parameters BEGIN -->
             <k>3742</k><!-- [N/m] spring constant -->
@@ -31,5 +29,5 @@
             <R_pretension>0.01</R_pretension><!-- [m] motor 2 spool radius -->
             <!-- Maccepa 2.0 parameters END -->
-            <joint_motor>elbow_motor_joint</joint_motor>
+            <cardioid_motor_joint>elbow_motor_joint</cardioid_motor_joint>
         </plugin>
     </gazebo>

File: maccepa_description/urdf/camdisk/maccepa_camdisk.urdf.xacro (robot description, xacro)
@@ -10,7 +10,8 @@
       </inertial>
       <visual>
-        <origin xyz="${length/2} 0 0" rpy="0 0 0"/>
+        <!--<origin xyz="${length/2} 0 0" rpy="0 0 0"/>-->
         <geometry>
-          <box size="${length} 0.005 0.005"/>
+          <!--<box size="${length} 0.005 0.005"/>-->
+          <mesh filename="package://maccepa_description/stl/camdisk.stl" scale="0.001 0.001 0.001"/>
         </geometry>
         <material name="${material}"/>

File: maccepa_description/urdf/materials.xacro (robot description, xacro)
@@ -19,5 +19,5 @@
                     <diffuse>${rgba}</diffuse>
                     <specular>0 0 0 0</specular>
-                    <emissive>${rgba}</emissive>
+                    <!--<emissive>${rgba}</emissive>-->
                 </material>
             </visual>
@@ -25,5 +25,5 @@
     </xacro:macro>
     <xacro:macro name="gazebo_green" params="reference">
-        <gazebo_emissive_color reference="${reference}" rgba="0.0 1.0 0.0 1"/>
+        <gazebo_emissive_color reference="${reference}" rgba="0.0 1.0 0.0 0.3"/>
     </xacro:macro>
     <xacro:macro name="gazebo_blue" params="reference">
@@ -36,3 +36,54 @@
         <gazebo_emissive_color reference="${reference}" rgba="1.0 1.0 0.0 1"/>
     </xacro:macro>
+    <xacro:macro name="gazebo_darkgreen" params="reference">
+        <gazebo_emissive_color reference="${reference}" rgba="0.47 0.87 0.47 0.5"/>
+    </xacro:macro>
+    <xacro:macro name="gazebo_darkblue" params="reference">
+        <gazebo_emissive_color reference="${reference}" rgba="0.0 0.19 0.33 1"/>
+    </xacro:macro>
+    <xacro:macro name="gazebo_crimson" params="reference">
+        <gazebo_emissive_color reference="${reference}" rgba="0.86 0.08 0.23 1"/>
+    </xacro:macro>
+    <xacro:macro name="gazebo_gold" params="reference">
+        <gazebo_emissive_color reference="${reference}" rgba="0.72 0.53 0.04 1"/>
+    </xacro:macro>
+    <xacro:macro name="contact_surface" params="reference">
+        <gazebo reference="${reference}">
+            <!-- for some reason none of these parameters don't apply in gazebo-->
+            <!--<collision>-->
+                <!--<surface>-->
+                    <!--<bounce>-->
+                        <!--<restitution_coefficient>0.0</restitution_coefficient>-->
+                    <!--</bounce>-->
+                    <!--<friction>-->
+                        <!--<torsional>&lt;!&ndash; works only with ODE &ndash;&gt;-->
+                            <!--<coefficient>1.0</coefficient>-->
+                            <!--<surface_radius>0.01</surface_radius>-->
+                            <!--<use_patch_radius>false</use_patch_radius>-->
+                        <!--</torsional>-->
+                        <!--<ode>-->
+                            <!--<mu>0.8</mu>-->
+                            <!--<mu2>0.8</mu2>-->
+                        <!--</ode>-->
+                    <!--</friction>-->
+                    <!--<contact>-->
+                        <!--<collide_without_contact>1</collide_without_contact>-->
+                        <!--<poissons_ratio>0.1</poissons_ratio>-->
+                        <!--<elastic_modulus>1</elastic_modulus>-->
+                        <!--<ode>-->
+                            <!--<kp>100000</kp>-->
+                            <!--<kd>1000.0</kd>-->
+                            <!--<max_vel>100000.0</max_vel>-->
+                            <!--<min_depth>0.001</min_depth>-->
+                        <!--</ode>-->
+                    <!--</contact>-->
+                <!--</surface>-->
+            <!--</collision>-->
+            <!-- while parameters set as follows apply -->
+            <minDepth value="0.01"/>
+            <maxVel value="0.0"/>
+            <mu1 value="0.8"/>
+            <mu2 value="0.8"/>
+        </gazebo>
+    </xacro:macro>
 </robot>
